File: kicad/kicad.sch (KiCad schematic (older format))
At the start: 34 parts

Commit message: Save progress on schematic.
Connections:
- net +5V: now also C?.1, U?.1 (1~CLR), U?.10 (CET), U?.14 (VCC), U?.16 (VCC), U?.16 (VCC), U?.16 (VCC), U?.16 (VCC), U?.4 (1~PRE), U?.7 (CEP), U?.9 (~PE), U?.9 (~PE), U?.9 (~PE), U?.9 (~PE), U?.9 (~PE), X?.8 (Vcc)
- net GND: now also C?.2, U?.7 (GND), U?.8 (GND), U?.8 (GND), U?.8 (GND), U?.8 (GND), X?.4 (GND)
- net at U?.11 (P4), U?.11 (Q3): now also U?.5 (I0b) (x2)
- net at U?.12 (Q2), U?.13 (P5): now also U?.2 (I0a) (x2)
- net at U?.13 (Q1), U?.15 (P6): now also U?.11 (I0c) (x2)
- net at U?.14 (Q0), U?.17 (P7): now also U?.14 (I0d) (x2)
- net at U?.11 (Q3), U?.2 (P0): now also U?.5 (I0b) (x2)
- net at U?.12 (Q2), U?.4 (P1): now also U?.2 (I0a) (x2)
- net at U?.13 (Q1), U?.6 (P2): now also U?.11 (I0c) (x2)
- net at U?.14 (Q0), U?.8 (P3): now also U?.14 (I0d) (x2)
- net at U?.10 (3B): now also U?.12 (6Y)
- net at U?.2 (1B): now also U?.8 (3Y)
- net at U?.3 (1Y): now also U?.1 (~MR), U?.1 (~MR), U?.1 (~MR), U?.1 (~MR), U?.1 (~MR)
- net at U?.4 (2A): now also U?.6 (I1b)
- net at U?.5 (2B): now also U?.8 (4Y)
- net at U?.6 (2Y): now also U?.1 (1A)
- net at U?.9 (3A): now also U?.10 (5Y)
- net at U?.2 (1D): now also U?.6 (1~Q)
- net at U?.3 (1CLK): now also X?.5 (OUT)
- net at U?.5 (1Q): now also U?.2 (CP), U?.2 (CP), U?.2 (CP), U?.2 (CP), U?.2 (CP)
- net at U?.15 (TC): now also U?.10 (CET), U?.7 (CEP) (x4)
- net at U?.13 (Q1): now also U?.11 (5A), U?.11 (I0c)
- net at U?.14 (Q0): now also U?.13 (6A), U?.14 (I0d)

Commit message: Save progress on schematic.
Parts:
- added J?: Address In, symbol Connector:Conn_01x18_Male
- added J?: Mode In, symbol Connector:Conn_01x02_Male
- added J?: Data In, symbol Connector:Conn_01x05_Male
- added J?: VGA Out, symbol Connector:Conn_01x05_Male
- added J?: Power, symbol Connector:Conn_01x05_Male
- added J?: L77HDE15SD1CH4F, AMPHENOL_L77HDE15SD1CH4F, symbol L77HDE15SD1CH4F:L77HDE15SD1CH4F
Connections:
- net +5V: now also U?.10 (2~PRE), U?.13 (2~CLR), U?.14 (VCC), U?.14 (VCC), U?.16 (VCC), U?.16 (VCC), U?.16 (VCC), U?.16 (VCC), U?.16 (VCC), U?.16 (VCC), U?.16 (VCC), U?.16 (VCC), U?.16 (VCC), U?.16 (VCC), U?.2 (I0a), U?.2 (I0a)
- net GND: now also U?.15 (E), U?.15 (E), U?.15 (E), U?.15 (E), U?.15 (E), U?.15 (E), U?.15 (E), U?.15 (E), U?.15 (E), U?.15 (E), U?.5 (I0b), U?.5 (I0b), U?.7 (GND), U?.7 (GND), U?.8 (GND), U?.8 (GND), U?.8 (GND), U?.8 (GND), U?.8 (GND), U?.8 (GND), U?.8 (GND), U?.8 (GND), U?.8 (GND), U?.8 (GND)
- net at U?.11 (P4), U?.11 (Q3), U?.5 (I0b): now also U?.5 (I0b) (x2)
- net at U?.12 (Q2), U?.13 (P5), U?.2 (I0a): now also U?.2 (I0a) (x2)
- net at U?.11 (I0c), U?.13 (Q1), U?.15 (P6): now also U?.11 (I0c) (x2)
- net at U?.14 (I0d), U?.14 (Q0), U?.17 (P7): now also U?.14 (I0d) (x2)
- net at U?.11 (Q3), U?.2 (P0), U?.5 (I0b): now also U?.5 (I0b) (x2)
- net at U?.12 (Q2), U?.2 (I0a), U?.4 (P1): now also U?.2 (I0a) (x2)
- net at U?.11 (I0c), U?.13 (Q1), U?.6 (P2): now also U?.11 (I0c) (x2)
- net at U?.14 (I0d), U?.14 (Q0), U?.8 (P3): now also U?.14 (I0d) (x2)
- net at U?.4 (2A), U?.6 (I1b): now also U?.6 (I1b)
- net at U?.11 (5A), U?.11 (I0c), U?.13 (Q1): now also U?.11 (I0c)
- net at U?.13 (6A), U?.14 (I0d), U?.14 (Q0): now also U?.14 (I0d)
- net at U?.2 (1Y): now also U?.11 (2CLK)
- net at U?.9 (4A): now also U?.3 (I1a), U?.3 (I1a)
- net at U?.1 (S): now also U?.1 (S), U?.1 (S), U?.1 (S), U?.1 (S), U?.24 (OE), U?.9 (2Q)
- net at U?.10 (I1c): now also U?.10 (I1c), J?.2 (Pin_2)
- net at U?.12 (Zd): now also U?.12 (A0) (x2)
- net at U?.13 (I1d): now also U?.13 (I1d), J?.1 (Pin_1)
- net at U?.3 (I1a): now also U?.3 (I1a), J?.3 (Pin_3)
- net at U?.4 (Za): now also U?.10 (A2) (x2)
- net at U?.6 (I1b): now also U?.6 (I1b), J?.4 (Pin_4)
- net at U?.7 (Zb): now also U?.9 (A3) (x2)
- net at U?.9 (Zc): now also U?.11 (A1) (x2)
- net at U?.10 (I1c): now also U?.10 (I1c) (x4)
- net at U?.12 (Zd): now also U?.8 (A4) (x2)
- net at U?.13 (I1d): now also U?.13 (I1d) (x4)
- net at U?.3 (I1a): now also U?.3 (I1a) (x3)
- net at U?.4 (Za): now also U?.6 (A6) (x2)
- net at U?.6 (I1b): now also U?.6 (I1b) (x3)
- net at U?.7 (Zb): now also U?.5 (A7) (x2)
- net at U?.9 (Zc): now also U?.7 (A5) (x2)
- net at U?.12 (Zd): now also U?.27 (A8) (x2)
- net at U?.4 (Za): now also U?.23 (A10) (x2)
- net at U?.7 (Zb): now also U?.25 (A11) (x2)
- net at U?.9 (Zc): now also U?.26 (A9) (x2)
- net at U?.12 (Zd): now also U?.4 (A12) (x2)
- net at U?.4 (Za): now also U?.3 (A14) (x2)
- net at U?.7 (Zb): now also U?.31 (A15) (x2)
- net at U?.9 (Zc): now also U?.28 (A13) (x2)
- net at U?.12 (Zd): now also U?.2 (A16) (x2)
- net at U?.4 (Za): now also U?.29 (WE) (x2)
- net at U?.7 (Zb): now also U?.22 (CE) (x2)
- net at U?.9 (Zc): now also U?.30 (A17) (x2)
- net at U?.1 (S): now also U?.1 (S), U?.1 (S), U?.1 (S), U?.1 (S), U?.12 (2D), U?.24 (OE), U?.8 (2~Q)
- new net: J?.S1 (SHIELD), J?.S2 (SHIELD)
Other:
- note added: "A0"
- note added: "CE"
- note added: "WE"

Commit message: Save progress on schematic.
Connections:
- net +5V: now also C?.1, J?.1 (Pin_1), J?.2 (Pin_2), U?.20 (VCC), U?.20 (VCC), U?.20 (VCC), U?.20 (VCC), U?.32 (VCC), U?.32 (VCC)
- net GND: now also C?.2, J?.10, J?.3 (Pin_3), J?.4 (Pin_4), J?.5, J?.5 (Pin_5), J?.6, J?.7, J?.8, U?.1 (A18), U?.1 (A18), U?.10 (GND), U?.10 (GND), U?.10 (GND), U?.10 (GND), U?.16 (VSS), U?.16 (VSS)
- net at U?.4 (2A), U?.6 (I1b), U?.6 (I1b): now also J?.2 (Pin_2)
- net at U?.3 (I1a), U?.3 (I1a), U?.9 (4A): now also J?.1 (Pin_1)
- net at U?.1 (S), U?.1 (S), U?.1 (S)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: now also U?.1 (1~G), U?.1 (1~G), U?.19 (2~G/2G+), U?.19 (2~G/2G+)
- net at U?.10 (I1c), U?.10 (I1c): now also J?.6 (Pin_6)
- net at U?.13 (I1d), U?.13 (I1d): now also J?.5 (Pin_5)
- net at U?.3 (I1a), U?.3 (I1a): now also J?.7 (Pin_7)
- net at U?.6 (I1b), U?.6 (I1b): now also J?.8 (Pin_8)
- net at U?.10 (I1c), U?.10 (I1c): now also J?.10 (Pin_10)
- net at U?.13 (I1d), U?.13 (I1d): now also J?.9 (Pin_9)
- net at U?.3 (I1a), U?.3 (I1a): now also J?.11 (Pin_11)
- net at U?.6 (I1b), U?.6 (I1b): now also J?.12 (Pin_12)
- net at U?.10 (I1c), U?.10 (I1c): now also J?.14 (Pin_14)
- net at U?.13 (I1d), U?.13 (I1d): now also J?.13 (Pin_13)
- net at U?.3 (I1a), U?.3 (I1a): now also J?.15 (Pin_15)
- net at U?.6 (I1b), U?.6 (I1b): now also J?.16 (Pin_16)
- net at U?.10 (I1c), U?.10 (I1c): now also J?.18 (Pin_18)
- net at U?.13 (I1d), U?.13 (I1d): now also J?.17 (Pin_17)
- net at U?.1 (S), U?.1 (S), U?.1 (S)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: now also U?.1 (1~G), U?.1 (1~G), U?.19 (2~G/2G+), U?.19 (2~G/2G+)
- net at U?.11 (2A1): now also U?.18 (DQ4), U?.9 (2Y1) (x2)
- net at U?.12 (1Y4): now also J?.13, J?.4 (Pin_4), U?.12 (1Y4)
- net at U?.14 (1Y3): now also J?.3, J?.3 (Pin_3), U?.14 (1Y3)
- net at U?.16 (1Y2): now also J?.2, J?.2 (Pin_2), U?.16 (1Y2)
- net at U?.18 (1Y1): now also J?.1, J?.1 (Pin_1), U?.18 (1Y1)
- net at U?.2 (1A1): now also U?.13 (DQ0), U?.18 (1Y1) (x2)
- net at U?.4 (1A2): now also U?.14 (DQ1), U?.16 (1Y2) (x2)
- net at U?.6 (1A3): now also U?.14 (1Y3), U?.15 (DQ2) (x2)
- net at U?.8 (1A4): now also U?.12 (1Y4), U?.17 (DQ3) (x2)
- net at U?.9 (2Y1): now also J?.14, J?.5 (Pin_5), U?.9 (2Y1)
- net at U?.11 (2A1): now also J?.5 (Pin_5), U?.11 (2A1)
- net at U?.2 (1A1): now also J?.1 (Pin_1), U?.2 (1A1)
- net at U?.4 (1A2): now also J?.2 (Pin_2), U?.4 (1A2)
- net at U?.6 (1A3): now also J?.3 (Pin_3), U?.6 (1A3)
- net at U?.8 (1A4): now also J?.4 (Pin_4), U?.8 (1A4)
Other:
- note added: "B"
- note added: "D0"
- note added: "G"
- note added: "H"
- note added: "R"
- note added: "V"
- moved on the sheet: J?, U?

Commit message: Save progress on schematic.
Parts:
- added R? (x3): 200, symbol Device:R
- added R? (x3): 100, symbol Device:R
Connections:
- net GND: now also R?.1, R?.2, R?.2
- net at U?.14 (1Y3), U?.14 (1Y3): now also R?.1; no longer J?.3, J?.3 (Pin_3)
- net at U?.16 (1Y2), U?.16 (1Y2): now also R?.1; no longer J?.2, J?.2 (Pin_2)
- net at U?.18 (1Y1), U?.18 (1Y1): now also R?.1; no longer J?.1, J?.1 (Pin_1)
- new net: J?.1, J?.1 (Pin_1), R?.1, R?.2
- new net: J?.2, J?.2 (Pin_2), R?.1, R?.2
- new net: J?.3, J?.3 (Pin_3), R?.2, R?.2
Other:
- moved on the sheet: J?
Changed lines of the file:
@@
 L Connector:Conn_01x05_Male J?
 U 1 1 634892F6
-P 20900 17550
-F 0 "J?" V 21054 17262 50  0000 R CNN
-F 1 "VGA Out" V 20963 17262 50  0000 R CNN
-F 2 "" H 20900 17550 50  0001 C CNN
-F 3 "~" H 20900 17550 50  0001 C CNN
-	1    20900 17550
+P 19700 17900
+F 0 "J?" V 19854 17612 50  0000 R CNN
+F 1 "VGA Out" V 19763 17612 50  0000 R CNN
+F 2 "" H 19700 17900 50  0001 C CNN
+F 3 "~" H 19700 17900 50  0001 C CNN
+	1    19700 17900
 	0    -1   -1   0
 $EndComp
@@
 	1    0    0    -1
 $EndComp
-Text Notes 20700 17650 0    50   ~ 0
+Text Notes 19500 18000 0    50   ~ 0
 R
-Text Notes 20800 17650 0    50   ~ 0
+Text Notes 19600 18000 0    50   ~ 0
 G
-Text Notes 20900 17650 0    50   ~ 0
+Text Notes 19700 18000 0    50   ~ 0
 B
-Text Notes 21000 17650 0    50   ~ 0
+Text Notes 19800 18000 0    50   ~ 0
 H
-Text Notes 21100 17650 0    50   ~ 0
+Text Notes 19900 18000 0    50   ~ 0
 V
 $Comp
@@
 	22700 15850 20700 15850
 Wire Wire Line
-	20700 15850 20700 16350
-Wire Wire Line
 	22650 13300 22650 15900
 Wire Wire Line
 	22650 15900 20800 15900
 Wire Wire Line
-	20800 15900 20800 16500
-Wire Wire Line
 	22450 13400 22600 13400
 Wire Wire Line
@@
 	22600 15950 20900 15950
 Wire Wire Line
-	20900 15950 20900 16700
-Wire Wire Line
 	22450 13500 22550 13500
 Wire Wire Line
@@
 	22550 16000 21000 16000
 Wire Wire Line
-	21000 16000 21000 17150
-Wire Wire Line
 	22450 13700 22500 13700
 Wire Wire Line
@@
 Wire Wire Line
 	22500 16050 21100 16050
-Wire Wire Line
-	21100 16050 21100 17300
 Wire Wire Line
 	20300 8350 20700 8350
@@
 	20300 8750 20450 8750
 Wire Wire Line
-	20700 16350 22250 16350
-Wire Wire Line
-	22250 16350 22250 16200
-Wire Wire Line
-	22250 16200 22750 16200
-Wire Wire Line
 	1150 18150 25000 18150
-Connection ~ 20700 16350
-Wire Wire Line
-	20700 16350 20700 17350
-Wire Wire Line
-	20800 16500 22350 16500
-Wire Wire Line
-	22350 16500 22350 16300
-Wire Wire Line
-	22350 16300 22750 16300
-Connection ~ 20800 16500
-Wire Wire Line
-	20800 16500 20800 17350
-Wire Wire Line
-	20900 16700 22500 16700
-Wire Wire Line
-	22500 16700 22500 16400
-Wire Wire Line
-	22500 16400 22750 16400
-Connection ~ 20900 16700
-Wire Wire Line
-	20900 16700 20900 17350
-Wire Wire Line
-	21000 17150 22150 17150
-Wire Wire Line
-	22150 17150 22150 17600
-Wire Wire Line
-	22150 17600 22750 17600
-Connection ~ 21000 17150
-Wire Wire Line
-	21000 17150 21000 17350
-Wire Wire Line
-	21100 17300 22000 17300
-Wire Wire Line
-	22000 17300 22000 17700
-Wire Wire Line
-	22000 17700 22750 17700
-Connection ~ 21100 17300
-Wire Wire Line
-	21100 17300 21100 17350
 $Comp
 L power:GND #PWR?
@@
 	0    1    1    0
 $EndComp
+Wire Wire Line
+	20700 15850 20700 17350
+$Comp
+L Device:R R?
+U 1 1 671DFF81
+P 19150 17100
+F 0 "R?" H 19220 17146 50  0000 L CNN
+F 1 "200" H 19220 17055 50  0000 L CNN
+F 2 "" V 19080 17100 50  0001 C CNN
+F 3 "~" H 19150 17100 50  0001 C CNN
+	1    19150 17100
+	1    0    0    -1
+$EndComp
+$Comp
+L Device:R R?
+U 1 1 672CE19D
+P 19400 17100
+F 0 "R?" H 19470 17146 50  0000 L CNN
+F 1 "200" H 19470 17055 50  0000 L CNN
+F 2 "" V 19330 17100 50  0001 C CNN
+F 3 "~" H 19400 17100 50  0001 C CNN
+	1    19400 17100
+	1    0    0    -1
+$EndComp
+$Comp
+L Device:R R?
+U 1 1 672CEC76
+P 19650 17100
+F 0 "R?" H 19720 17146 50  0000 L CNN
+F 1 "200" H 19720 17055 50  0000 L CNN
+F 2 "" V 19580 17100 50  0001 C CNN
+F 3 "~" H 19650 17100 50  0001 C CNN
+	1    19650 17100
+	1    0    0    -1
+$EndComp
+Wire Wire Line
+	19150 17250 19150 17450
+Wire Wire Line
+	19150 17700 19500 17700
+Wire Wire Line
+	19400 17500 19600 17500
+Wire Wire Line
+	19600 17500 19600 17700
+Wire Wire Line
+	19650 17250 19650 17300
+Wire Wire Line
+	19650 17500 19700 17500
+Wire Wire Line
+	19700 17500 19700 17700
+Wire Wire Line
+	20700 17350 20400 17350
+Wire Wire Line
+	20400 17350 20400 16550
+Wire Wire Line
+	20400 16550 19150 16550
+Wire Wire Line
+	19150 16550 19150 16950
+Wire Wire Line
+	20800 17400 20350 17400
+Wire Wire Line
+	20350 17400 20350 16600
+Wire Wire Line
+	20350 16600 19400 16600
+Wire Wire Line
+	19400 16600 19400 16950
+Wire Wire Line
+	20800 15900 20800 17400
+Wire Wire Line
+	20900 17450 20300 17450
+Wire Wire Line
+	20300 17450 20300 16650
+Wire Wire Line
+	20300 16650 19650 16650
+Wire Wire Line
+	19650 16650 19650 16950
+Wire Wire Line
+	20900 15950 20900 17450
+Wire Wire Line
+	21000 17550 19800 17550
+Wire Wire Line
+	19800 17550 19800 17700
+Wire Wire Line
+	21000 16000 21000 17550
+Wire Wire Line
+	21100 17700 19900 17700
+Wire Wire Line
+	21100 16050 21100 17700
+$Comp
+L Device:R R?
+U 1 1 67A61F3B
+P 19000 17450
+F 0 "R?" V 18793 17450 50  0000 C CNN
+F 1 "100" V 18884 17450 50  0000 C CNN
+F 2 "" V 18930 17450 50  0001 C CNN
+F 3 "~" H 19000 17450 50  0001 C CNN
+	1    19000 17450
+	0    1    1    0
+$EndComp
+Connection ~ 19150 17450
+Wire Wire Line
+	19150 17450 19150 17600
+$Comp
+L Device:R R?
+U 1 1 67A62A68
+P 19800 17300
+F 0 "R?" V 19593 17300 50  0000 C CNN
+F 1 "100" V 19684 17300 50  0000 C CNN
+F 2 "" V 19730 17300 50  0001 C CNN
+F 3 "~" H 19800 17300 50  0001 C CNN
+	1    19800 17300
+	0    1    1    0
+$EndComp
+Connection ~ 19650 17300
+Wire Wire Line
+	19650 17300 19650 17500
+$Comp
+L Device:R R?
+U 1 1 67A6355B
+P 18750 17750
+F 0 "R?" V 18543 17750 50  0000 C CNN
+F 1 "100" V 18634 17750 50  0000 C CNN
+F 2 "" V 18680 17750 50  0001 C CNN
+F 3 "~" H 18750 17750 50  0001 C CNN
+	1    18750 17750
+	0    1    1    0
+$EndComp
+Wire Wire Line
+	18900 17750 19400 17750
+Wire Wire Line
+	19400 17250 19400 17350
+Connection ~ 19400 17500
+Wire Wire Line
+	19400 17500 19400 17750
+$Comp
+L power:GND #PWR?
+U 1 1 67B5C404
+P 18850 17450
+F 0 "#PWR?" H 18850 17200 50  0001 C CNN
+F 1 "GND" V 18855 17322 50  0000 R CNN
+F 2 "" H 18850 17450 50  0001 C CNN
+F 3 "" H 18850 17450 50  0001 C CNN
+	1    18850 17450
+	0    1    1    0
+$EndComp
+$Comp
+L power:GND #PWR?
+U 1 1 67B5CCA7
+P 18600 17750
+F 0 "#PWR?" H 18600 17500 50  0001 C CNN
+F 1 "GND" V 18605 17622 50  0000 R CNN
+F 2 "" H 18600 17750 50  0001 C CNN
+F 3 "" H 18600 17750 50  0001 C CNN
+	1    18600 17750
+	0    1    1    0
+$EndComp
+$Comp
+L power:GND #PWR?
+U 1 1 67B5D566
+P 19950 17300
+F 0 "#PWR?" H 19950 17050 50  0001 C CNN
+F 1 "GND" V 19955 17172 50  0000 R CNN
+F 2 "" H 19950 17300 50  0001 C CNN
+F 3 "" H 19950 17300 50  0001 C CNN
+	1    19950 17300
+	0    -1   -1   0
+$EndComp
+Wire Wire Line
+	21000 17550 22400 17550
+Wire Wire Line
+	22400 17550 22400 17600
+Wire Wire Line
+	22400 17600 22750 17600
+Connection ~ 21000 17550
+Wire Wire Line
+	21100 17700 22750 17700
+Connection ~ 21100 17700
+Wire Wire Line
+	19150 17600 18650 17600
+Wire Wire Line
+	18650 17600 18650 16200
+Wire Wire Line
+	18650 16200 22750 16200
+Connection ~ 19150 17600
+Wire Wire Line
+	19150 17600 19150 17700
+Wire Wire Line
+	19400 17350 18700 17350
+Wire Wire Line
+	18700 17350 18700 16300
+Wire Wire Line
+	18700 16300 22750 16300
+Connection ~ 19400 17350
+Wire Wire Line
+	19400 17350 19400 17500
+Wire Wire Line
+	19700 17500 21150 17500
+Wire Wire Line
+	21150 17500 21150 16400
+Wire Wire Line
+	21150 16400 22750 16400
+Connection ~ 19700 17500
 $EndSCHEMATC

Commit message: Save progress on schematic.
Parts:
- C1, C2, C3: renamed from C?; footprint (none) -> Capacitor_THT:CP_Radial_D10.0mm_P5.00mm
- J1, J7, J9: renamed from J?; footprint (none) -> Connector_PinHeader_2.54mm:PinHeader_1x05_P2.54mm_Vertical
- J2: renamed from J?; footprint (none) -> Connector_PinHeader_2.54mm:PinHeader_1x18_P2.54mm_Vertical
- J3, J4, J6: renamed from J?; footprint (none) -> Connector_PinHeader_2.54mm:PinHeader_1x16_P2.54mm_Vertical
- J5: renamed from J?; footprint (none) -> Connector_PinHeader_2.54mm:PinHeader_1x02_P2.54mm_Vertical
- J8: renamed from J?; footprint AMPHENOL_L77HDE15SD1CH4F -> L77HDE15SD1CH4F:AMPHENOL_L77HDE15SD1CH4F
- R1, R2, R3, R4, R5, R6: renamed from R?; footprint (none) -> Resistor_THT:R_Axial_DIN0207_L6.3mm_D2.5mm_P7.62mm_Horizontal
- U1, U11, U12, U13, U14, U15, U16, U17, U19, U2, U5, U6, U7, U8, U9: renamed from U?; footprint (none) -> Package_DIP:DIP-16_W7.62mm
- U10, U4: renamed from U?; footprint N20 -> Package_DIP:DIP-20_W7.62mm
- U18, U20, U22, U3: renamed from U?; footprint DIP794W45P254L1969H508Q14 -> Package_DIP:DIP-14_W7.62mm
- U21, U23: renamed from U?; footprint DIP254P1524X393-32 -> Package_DIP:DIP-32_W15.24mm
- U24, U25, U26, U27: renamed from U?; footprint DIP254P762X508-20 -> Package_DIP:DIP-20_W7.62mm
- gave numbers to parts that had none: 1
