File: kicad/kicad.kicad_pcb (KiCad board)
At the start: 2 copper layers, 46 parts, among them J1 Power, J2 Address In, J3 Counter Reset Value, J4 5V, J5 Mode In, J6 GND, J7 VGA Out, J8 L77HDE15SD1CH4F, J9 Data In, U1 74LS157, U10 SN74LS682N, U11 74LS161, U12 74LS157, U13 74LS157, U14 74LS161, U15 74LS157, U16 74LS157, U17 74LS161, U18 SN74HC32N, U19 74LS161, U2 74LS157, U20 SN74LS04N, U21 AS6C4008-55PCN, U22 SN74LS74AN, U23 AS6C4008-55PCN, U24 SN74LS244N, U25 SN74LS244N, U26 SN74LS244N, U27 SN74LS244N, U3 SN74LS74AN, U4 SN74LS682N, U5 74LS157, U6 74LS157, U7 74LS161, U8 74LS157, U9 74LS157, X1 CXO_DIP8

Commit message: Save progress on PCB.
Parts:
- moved J6 126.3 mm to (315.4, 164.5), turned to 90 degrees
- moved J3 108.6 mm to (315.4, 162.0), turned to 90 degrees
- moved J4 91.5 mm to (315.4, 159.5), turned to 90 degrees
- moved U22 73.2 mm to (380.8, 184.2)
- moved U20 66.7 mm to (367.4, 184.3)
- moved U19 55.6 mm to (354.8, 184.1)
- moved U18 51.1 mm to (365.2, 162.0)
- moved U17 45.3 mm to (342.7, 184.2)
- moved U10 41.3 mm to (359.8, 170.0), turned to 270 degrees
- moved U4 37.2 mm to (330.3, 170.0), turned to 270 degrees
- moved U14 34.0 mm to (330.6, 184.2)
- moved X1 24.8 mm to (285.8, 197.0)
- moved U11 22.4 mm to (319.3, 184.2)
- moved U7 11.9 mm to (307.9, 184.2)

Commit message: Save progress on PCB.
Parts:
- moved C2 214.8 mm to (361.2, 159.9)
- moved J8 191.3 mm to (358.9, 246.7)
- moved C1 170.4 mm to (284.9, 161.1)
- moved J9 152.8 mm to (420.1, 207.4)
- moved J7 141.6 mm to (364.1, 238.3), turned to 270 degrees
- moved R1 136.2 mm to (339.3, 248.1), turned to 180 degrees
- moved R6 125.1 mm to (331.7, 251.4)
- moved J1 121.9 mm to (282.2, 250.0), turned to 180 degrees
- moved R5 115.8 mm to (383.9, 234.8)
- moved R4 109.6 mm to (404.7, 234.8), turned to 180 degrees
- moved C3 103.8 mm to (287.6, 244.8)
- moved R3 102.8 mm to (391.5, 231.5), turned to 180 degrees
- moved J5 101.9 mm to (420.1, 223.3)
- moved R2 97.4 mm to (339.3, 254.8), turned to 180 degrees
- moved J2 84.7 mm to (282.2, 254.9), turned to 90 degrees
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Routing:
- added copper zone on PWR, net +5V
- added copper zone on GND, net GND
Other:
- board outline added: 147.3 x 104.8 mm
- copper layers 2 -> 4

Commit message: Save progress on PCB.
Parts:
- moved C2 1.05 mm to (360.3, 159.4)
Routing:
- net Net-(U18-Pad13): track 0.00 -> 69.7 mm, vias 0 -> 2
- net Net-(J3-Pad3): track 0.00 -> 41.7 mm, vias 0 -> 2
- net Net-(J3-Pad4): track 0.00 -> 40.6 mm
- net Net-(J3-Pad9): track 0.00 -> 40.6 mm, vias 0 -> 2
- net Net-(J3-Pad2): track 0.00 -> 36.1 mm, vias 0 -> 2
- net Net-(U11-Pad14): track 0.00 -> 35.3 mm, vias 0 -> 1
- net Net-(J3-Pad1): track 0.00 -> 34.2 mm, vias 0 -> 2
- net Net-(J3-Pad10): track 0.00 -> 33.1 mm, vias 0 -> 2
- net Net-(U11-Pad13): track 0.00 -> 30.5 mm, vias 0 -> 2
- net Net-(U11-Pad12): track 0.00 -> 28.2 mm, vias 0 -> 1
- net Net-(U11-Pad11): track 0.00 -> 28.2 mm
- net Net-(U1-Pad5): track 0.00 -> 27.1 mm, vias 0 -> 1
- net Net-(J3-Pad11): track 0.00 -> 25.3 mm, vias 0 -> 2
- net Net-(U1-Pad2): track 0.00 -> 19.7 mm, vias 0 -> 1
- net Net-(J3-Pad12): track 0.00 -> 19.2 mm
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
Commit message: Save progress on PCB.
Routing:
- net Net-(U13-Pad1): track 0.00 -> 221.5 mm, vias 0 -> 4
- net Net-(U23-Pad6): track 0.00 -> 170.5 mm, vias 0 -> 2
- net Net-(U2-Pad9): track 0.00 -> 168.2 mm, vias 0 -> 2
- net Net-(U2-Pad4): track 0.00 -> 166.8 mm, vias 0 -> 1
- net Net-(U2-Pad7): track 0.00 -> 161.5 mm, vias 0 -> 2
- net Net-(U2-Pad12): track 0.00 -> 153.7 mm, vias 0 -> 1
- net Net-(U23-Pad5): track 0.00 -> 151.5 mm, vias 0 -> 2
- net Net-(U23-Pad7): track 0.00 -> 142.3 mm, vias 0 -> 2
- net Net-(U23-Pad8): track 0.00 -> 139.6 mm, vias 0 -> 2
- net Net-(U13-Pad4): track 0.00 -> 121.5 mm, vias 0 -> 2
- net Net-(J5-Pad2): track 0.00 -> 119.6 mm, vias 0 -> 1
- net Net-(U13-Pad7): track 0.00 -> 116.2 mm, vias 0 -> 4
- net Net-(U23-Pad23): track 0.00 -> 112.7 mm, vias 0 -> 2
- net Net-(U23-Pad27): track 0.00 -> 111.3 mm, vias 0 -> 1
- net Net-(U13-Pad12): track 0.00 -> 105.5 mm, vias 0 -> 2
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
Commit message: Save progress on PCB.
Routing:
- net Net-(U1-Pad1): track 0.00 -> 239.2 mm, vias 0 -> 7
- net Net-(U1-Pad12): track 0.00 -> 186.1 mm
- net Net-(U1-Pad9): track 0.00 -> 146.4 mm, vias 0 -> 1
- net Net-(U1-Pad4): track 0.00 -> 143.5 mm, vias 0 -> 1
- net Net-(U1-Pad7): track 0.00 -> 134.0 mm, vias 0 -> 2
- net Net-(J7-Pad3): track 24.3 -> 148.7 mm
- net Net-(U21-Pad13): track 0.00 -> 120.9 mm, vias 0 -> 7
- net Net-(U21-Pad8): track 0.00 -> 118.6 mm, vias 0 -> 2
- net Net-(J2-Pad18): track 13.0 -> 127.8 mm, vias 0 -> 4
- net Net-(J7-Pad4): track 0.00 -> 113.3 mm, vias 0 -> 3
- net Net-(U21-Pad6): track 0.00 -> 110.7 mm, vias 0 -> 3
- net Net-(U21-Pad7): track 0.00 -> 109.6 mm, vias 0 -> 2
- net Net-(J7-Pad5): track 0.00 -> 104.9 mm, vias 0 -> 4
- net Net-(J7-Pad2): track 37.1 -> 139.3 mm
- net Net-(U21-Pad5): track 0.00 -> 101.0 mm, vias 0 -> 4
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
Commit message: Save progress on PCB.
Other:
- board text added: "+5V"
- board text added: "100"
- board text added: "200"
- board text added: "25.175 MHz"
- board text added: "5V"
- board text added: "7404"
- board text added: "74157"
- board text added: "74161"
- board text added: "74244"
- board text added: "7432"
- board text added: "74682"
- board text added: "7474"
- board text added: "A0"
- board text added: "AS6C4008-55PCN"
- board text added: "Address In"
- board text added: "B"
- board text added: "CE"
- board text added: "Counter Reset Value"
- board text added: "D0"
- board text added: "Data In"
- board text added: "Default: HHHH LLHL LLHL HHLL"
- board text added: "G"
- board text added: "GND"
- board text added: "HS"
- board text added: "Mode In"
- board text added: "Nick Bild February 2022 github.com/nickbild/vectron_vga_plus_v2"
- board text added: "Power"
- board text added: "R"
- board text added: "VGA Out"
- board text added: "VS"
- board text added: "Vectron VGA Plus"
- board text added: "WE"
- board text added: "v2.0"

Commit message: Save progress on PCB.
Routing:
- net GND: track 0.00 -> 11.2 mm, vias 0 -> 1
